File: First_Crack_Controller.kicad_pcb (KiCad board)
At the start: 2 copper layers, 38 parts, among them J1 Conn_01x03, J12 TB006-508-02BE, J13 TB006-508-02BE, J2 24V input, J3 SM04B-SRSS-TB_LF__SN_, J4 SM04B-SRSS-TB_LF__SN_, J5 Conn_01x10, J8 Drum Connector, Q1 BSS138, Q2 BSS138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

Commit message: pcb board
Parts:
- J5: footprint Connector_Molex:Molex_PicoBlade_53047-1010_1x10_P1.25mm_Vertical -> Connector_PinHeader_2.54mm:PinHeader_1x10_P2.54mm_Vertical
- moved RV2 157.8 mm to (32.0, 29.0), turned to -90 degrees
- moved Q2 156.1 mm to (47.0, 27.0), turned to 180 degrees
- moved J3 149.6 mm to (19.0, 18.5), turned to -90 degrees
- moved J4 147.9 mm to (19.0, 28.5), turned to -90 degrees
- moved RV1 147.7 mm to (40.0, 29.0), turned to -90 degrees
- moved FB1 146.2 mm to (26.0, 38.6), turned to 90 degrees
- moved Q1 146.1 mm to (52.4, 32.0), turned to 180 degrees
- moved FB2 145.5 mm to (26.0, 43.6), turned to 90 degrees
- moved FB3 143.8 mm to (26.0, 51.6), turned to 90 degrees
- moved J1 143.2 mm to (34.5, 63.0), turned to -90 degrees
- moved FB4 143.2 mm to (26.0, 56.6), turned to 90 degrees
- moved R6 140.6 mm to (31.0, 38.6), turned to -90 degrees
- moved J2 139.6 mm to (77.8, 47.5)
- moved J8 139.6 mm to (77.8, 61.5)
- moved U4 139.2 mm to (66.3, 55.5)
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Connections:
- U1 pad 21: unconnected-(U1-EXP-Pad21) -> GND
- U2 pad 21: unconnected-(U2-EXP-Pad21) -> GND
- U3 pad 7: /KeyPad_INT -> unconnected-(U3-GPIO21_D6_TX-Pad7)
Routing:
- net GND: track 0.00 -> 345.0 mm, vias 0 -> 10
- net +5V: track 0.00 -> 181.9 mm, vias 0 -> 5
- net /Temp_Dial_Servo: track 0.00 -> 61.6 mm, vias 0 -> 2
- net +24V: track 0.00 -> 49.6 mm, vias 0 -> 4
- net /Drum_PWM_Reverse: track 0.00 -> 39.7 mm, vias 0 -> 2
- net /Drum_PWM_Forward: track 0.00 -> 38.5 mm, vias 0 -> 2
- net +3V3: track 0.00 -> 34.7 mm, vias 0 -> 5
- net /SCL5V: track 0.00 -> 28.6 mm, vias 0 -> 4
- net /SDA5V: track 0.00 -> 28.2 mm, vias 0 -> 4
- net /SCL3V3: track 0.00 -> 19.3 mm, vias 0 -> 2
- net /Display_Vo: track 0.00 -> 12.7 mm
- net /SDA3V3: track 0.00 -> 12.4 mm, vias 0 -> 3
- net Net-(U4-OUT1): track 0.00 -> 11.0 mm
- net /Display_Brightness: track 0.00 -> 10.7 mm
- net Net-(U5-IN): track 0.00 -> 10.5 mm, vias 0 -> 2
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Other:
- board outline added: 73 x 55 mm

Commit message: completed pcb
Routing:
- net /SDA5V: track 28.2 -> 92.8 mm, vias 4 -> 7
- net /SCL5V: track 28.6 -> 85.1 mm, vias 4 -> 6
- net GND: track 345.0 -> 356.1 mm, vias 10 -> 9
- net +3V3: track 34.7 -> 44.0 mm, vias 5 -> 4
- net +5V: track 181.9 -> 184.5 mm
- net Net-(U4-ILIM): vias 3 -> 2
- net /SDA3V3: vias 3 -> 2
Other:
- board text added: "First Crack Coffee Roaster"
